File: farway_hacks.kicad_sch (KiCad schematic)
At the start: 15 parts, among them J1 Conn_01x04, J2_servo1 Conn_01x03, J4 Conn_01x03, U1 ESP32-WROOM-32

Commit message: Updated schematics and pcb editor
Parts:
- BZ1: footprint (none) -> Buzzer_Beeper:Buzzer_12x9.5RM7.6
- C1_10uF1, C2_22uF1: footprint (none) -> Capacitor_THT:C_Radial_D5.0mm_H5.0mm_P2.00mm
- C3_100nF1: footprint (none) -> Capacitor_THT:C_Disc_D5.0mm_W2.5mm_P5.00mm
- D1_GREEN1, D2_RED1: footprint (none) -> LED_THT:LED_D5.0mm
- J1: footprint (none) -> Connector_PinHeader_2.54mm:PinHeader_1x04_P2.54mm_Vertical
- J2_servo1, J4: footprint (none) -> Connector_PinHeader_2.54mm:PinHeader_1x03_P2.54mm_Vertical
- PowerInput1: footprint (none) -> Connector_PinHeader_2.54mm:PinHeader_1x02_P2.54mm_Vertical
- R1_220Ω1, R2_220Ω1, R3_10k1: footprint (none) -> Resistor_THT:R_Axial_DIN0207_L6.3mm_D2.5mm_P10.16mm_Horizontal
Connections:
- net GND: now also J1.4 (Pin_4); no longer J1.2 (Pin_2)
- net at J2_servo1.2 (Pin_2), R1_220Ω1.2, U1.16 (IO13): no longer U1.14 (IO12)
- net at U1.28 (IO17): now also J1.2 (Pin_2); no longer J1.4 (Pin_4)
- no-connect marks 27 -> 28
Other:
- moved on the sheet: R2_220Ω1
Changed lines of the file:
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@@
+	)
+	(junction
+		(at 199.39 116.84)
+		(diameter 0)
+		(color 0 0 0 0)
 	)
 	(junction
@@
 	)
 	(junction
-		(at 127 96.52)
-		(diameter 0)
-		(color 0 0 0 0)
-	)
-	(junction
-		(at 195.58 116.84)
-		(diameter 0)
-		(color 0 0 0 0)
-	)
-	(junction
 		(at 27.94 27.94)
 		(diameter 0)
@@
 	)
 	(no_connect
+		(at 124.46 101.6)
+	)
+	(no_connect
 		(at 139.7 101.6)
 	)
@@
 	(wire
 		(pts
-			(xy 132.08 39.37) (xy 224.79 39.37)
-		)
-		(stroke
-			(width 0)
-			(type default)
-		)
-	)
-	(wire
-		(pts
-			(xy 124.46 96.52) (xy 124.46 101.6)
+			(xy 129.54 39.37) (xy 224.79 39.37)
 		)
 		(stroke
@@
 	(wire
 		(pts
-			(xy 137.16 101.6) (xy 137.16 92.71)
-		)
-		(stroke
-			(width 0)
-			(type default)
-		)
-	)
-	(wire
-		(pts
 			(xy 59.69 116.84) (xy 95.25 116.84)
 		)
@@
 	(wire
 		(pts
-			(xy 137.16 92.71) (xy 199.39 92.71)
-		)
-		(stroke
-			(width 0)
-			(type default)
-		)
-	)
-	(wire
-		(pts
 			(xy 45.72 157.48) (xy 59.69 157.48)
 		)
@@
 	(wire
 		(pts
-			(xy 134.62 90.17) (xy 199.39 90.17)
-		)
-		(stroke
-			(width 0)
-			(type default)
-		)
-	)
-	(wire
-		(pts
-			(xy 132.08 97.79) (xy 132.08 59.69)
+			(xy 137.16 87.63) (xy 137.16 101.6)
 		)
 		(stroke
@@
 	(wire
 		(pts
-			(xy 195.58 116.84) (xy 219.71 116.84)
+			(xy 175.26 116.84) (xy 199.39 116.84)
 		)
 		(stroke
@@
 	(wire
 		(pts
-			(xy 175.26 116.84) (xy 195.58 116.84)
-		)
-		(stroke
-			(width 0)
-			(type default)
-		)
-	)
-	(wire
-		(pts
-			(xy 273.05 152.4) (xy 271.78 152.4)
+			(xy 199.39 116.84) (xy 219.71 116.84)
 		)
 		(stroke
@@
 	(wire
 		(pts
-			(xy 134.62 101.6) (xy 134.62 90.17)
-		)
-		(stroke
-			(width 0)
-			(type default)
-		)
-	)
-	(wire
-		(pts
 			(xy 265.43 16.51) (xy 265.43 46.99)
 		)
@@
 	(wire
 		(pts
-			(xy 129.54 97.79) (xy 132.08 97.79)
-		)
-		(stroke
-			(width 0)
-			(type default)
-		)
-	)
-	(wire
-		(pts
 			(xy 199.39 58.42) (xy 220.98 58.42)
 		)
@@
 	(wire
 		(pts
-			(xy 132.08 52.07) (xy 132.08 39.37)
+			(xy 129.54 52.07) (xy 129.54 39.37)
 		)
 		(stroke
@@
 	(wire
 		(pts
+			(xy 199.39 92.71) (xy 199.39 116.84)
+		)
+		(stroke
+			(width 0)
+			(type default)
+		)
+	)
+	(wire
+		(pts
 			(xy 224.79 39.37) (xy 228.6 39.37)
 		)
@@
 	(wire
 		(pts
-			(xy 124.46 96.52) (xy 127 96.52)
-		)
-		(stroke
-			(width 0)
-			(type default)
-		)
-	)
-	(wire
-		(pts
 			(xy 187.96 85.09) (xy 199.39 85.09)
 		)
@@
 	(wire
 		(pts
-			(xy 129.54 97.79) (xy 129.54 101.6)
+			(xy 129.54 59.69) (xy 129.54 101.6)
 		)
 		(stroke
@@
 	(wire
 		(pts
-			(xy 127 96.52) (xy 127 60.96)
-		)
-		(stroke
-			(width 0)
-			(type default)
-		)
-	)
-	(wire
-		(pts
-			(xy 195.58 87.63) (xy 195.58 116.84)
+			(xy 127 60.96) (xy 127 101.6)
 		)
 		(stroke
@@
 	(wire
 		(pts
+			(xy 199.39 87.63) (xy 137.16 87.63)
+		)
+		(stroke
+			(width 0)
+			(type default)
+		)
+	)
+	(wire
+		(pts
 			(xy 228.6 39.37) (xy 228.6 27.94)
 		)
@@
 	(wire
 		(pts
-			(xy 199.39 87.63) (xy 195.58 87.63)
+			(xy 199.39 90.17) (xy 134.62 90.17)
 		)
 		(stroke
@@
 	(wire
 		(pts
+			(xy 134.62 90.17) (xy 134.62 101.6)
+		)
+		(stroke
+			(width 0)
+			(type default)
+		)
+	)
+	(wire
+		(pts
 			(xy 27.94 27.94) (xy 27.94 52.07)
-		)
-		(stroke
-			(width 0)
-			(type default)
-		)
-	)
-	(wire
-		(pts
-			(xy 127 101.6) (xy 127 96.52)
 		)
 		(stroke
@@
 			)
 		)
-		(property "Footprint" ""
+		(property "Footprint" "Buzzer_Beeper:Buzzer_12x9.5RM7.6"
 			(at 250.825 34.29 90)
 			(hide yes)
@@
 			)
 		)
-		(property "Footprint" ""
+		(property "Footprint" "Connector_PinHeader_2.54mm:PinHeader_1x03_P2.54mm_Vertical"
 			(at 228.6 22.86 0)
 			(hide yes)
@@
 			)
 		)
-		(property "Footprint" ""
+		(property "Footprint" "Capacitor_THT:C_Radial_D5.0mm_H5.0mm_P2.00mm"
 			(at 36.5252 142.24 0)
 			(hide yes)
@@
 			)
 		)
-		(property "Footprint" ""
+		(property "Footprint" "Capacitor_THT:C_Disc_D5.0mm_W2.5mm_P5.00mm"
 			(at 96.2152 146.05 0)
 			(hide yes)
@@
 			)
 		)
-		(property "Footprint" ""
+		(property "Footprint" "Capacitor_THT:C_Radial_D5.0mm_H5.0mm_P2.00mm"
 			(at 60.6552 142.24 0)
 			(hide yes)
@@
 			)
 		)
-		(property "Footprint" ""
+		(property "Footprint" "Resistor_THT:R_Axial_DIN0207_L6.3mm_D2.5mm_P10.16mm_Horizontal"
 			(at 73.66 133.858 90)
 			(hide yes)
@@
 		(dnp no)
 		(property "Reference" "J2_servo1"
-			(at 224.7899 55.88 90)
+			(at 231.648 64.516 90)
 			(show_name no)
 			(do_not_autoplace no)
@@
 		)
 		(property "Value" "Conn_01x03"
-			(at 227.3299 55.88 90)
+			(at 229.616 65.532 90)
 			(show_name no)
 			(do_not_autoplace no)
@@
 			)
 		)
-		(property "Footprint" ""
+		(property "Footprint" "Connector_PinHeader_2.54mm:PinHeader_1x03_P2.54mm_Vertical"
 			(at 226.06 60.96 0)
 			(hide yes)
@@
 	(symbol
 		(lib_id "power:PWR_FLAG")
-		(at 273.05 152.4 0)
+		(at 271.78 152.4 0)
 		(unit 1)
 		(body_style 1)
@@
 		(fields_autoplaced yes)
 		(property "Reference" "#FLG02"
-			(at 273.05 150.495 0)
+			(at 271.78 150.495 0)
 			(hide yes)
 			(show_name no)
@@
 		)
 		(property "Value" "PWR_FLAG"
-			(at 273.05 147.32 0)
+			(at 271.78 147.32 0)
 			(show_name no)
 			(do_not_autoplace no)
@@
 		)
 		(property "Footprint" ""
-			(at 273.05 152.4 0)
+			(at 271.78 152.4 0)
 			(hide yes)
 			(show_name no)
@@
 		)
 		(property "Datasheet" ""
-			(at 273.05 152.4 0)
+			(at 271.78 152.4 0)
 			(hide yes)
 			(show_name no)
@@
 		)
 		(property "Description" "Special symbol for telling ERC where power comes from"
-			(at 273.05 152.4 0)
+			(at 271.78 152.4 0)
 			(hide yes)
 			(show_name no)
@@
 	(symbol
 		(lib_id "Device:R")
-		(at 132.08 55.88 0)
+		(at 129.54 55.88 0)
 		(unit 1)
 		(body_style 1)
@@
 		(fields_autoplaced yes)
 		(property "Reference" "R2_220Ω1"
-			(at 134.62 54.6099 0)
+			(at 132.08 54.6099 0)
 			(show_name no)
 			(do_not_autoplace no)
@@
 		)
 		(property "Value" "R"
-			(at 134.62 57.1499 0)
+			(at 132.08 57.1499 0)
 			(show_name no)
 			(do_not_autoplace no)
@@
 			)
 		)
-		(property "Footprint" ""
-			(at 130.302 55.88 90)
+		(property "Footprint" "Resistor_THT:R_Axial_DIN0207_L6.3mm_D2.5mm_P10.16mm_Horizontal"
+			(at 127.762 55.88 90)
 			(hide yes)
 			(show_name no)
@@
 		)
 		(property "Datasheet" ""
-			(at 132.08 55.88 0)
+			(at 129.54 55.88 0)
 			(hide yes)
 			(show_name no)
@@
 		)
 		(property "Description" "Resistor"
-			(at 132.08 55.88 0)
+			(at 129.54 55.88 0)
 			(hide yes)
 			(show_name no)
@@
 		(in_pos_files yes)
 		(dnp no)
-		(fields_autoplaced yes)
 		(property "Reference" "R1_220Ω1"
-			(at 129.54 40.6399 0)
+			(at 114.808 42.164 0)
 			(show_name no)
 			(do_not_autoplace no)
@@
 			)
 		)
-		(property "Footprint" ""
+		(property "Footprint" "Resistor_THT:R_Axial_DIN0207_L6.3mm_D2.5mm_P10.16mm_Horizontal"
 			(at 125.222 41.91 90)
 			(hide yes)
@@
 			)
 		)
-		(property "Footprint" ""
+		(property "Footprint" "Connector_PinHeader_2.54mm:PinHeader_1x02_P2.54mm_Vertical"
 			(at 27.94 189.23 0)
 			(hide yes)
@@
 			)
 		)
-		(property "Footprint" ""
+		(property "Footprint" "Connector_PinHeader_2.54mm:PinHeader_1x04_P2.54mm_Vertical"
 			(at 204.47 87.63 0)
 			(hide yes)
@@
 			)
 		)
-		(property "Footprint" ""
+		(property "Footprint" "LED_THT:LED_D5.0mm"
 			(at 214.63 16.51 0)
 			(hide yes)
@@
 		(dnp no)
 		(property "Reference" "D1_GREEN1"
-			(at 231.14 44.7675 0)
+			(at 217.932 44.958 0)
 			(show_name no)
 			(do_not_autoplace no)
@@
 		)
 		(property "Value" "LED"
-			(at 228.6 44.7675 0)
-			(show_name no)
-			(do_not_autoplace no)
-			(effects
-				(font
-					(size 1.27 1.27)
-				)
-			)
-		)
-		(property "Footprint" ""
+			(at 220.218 41.91 0)
+			(show_name no)
+			(do_not_autoplace no)
+			(effects
+				(font
+					(size 1.27 1.27)
+				)
+			)
+		)
+		(property "Footprint" "LED_THT:LED_D5.0mm"
 			(at 224.79 43.18 0)
 			(hide yes)
