File: farway_hacks.kicad_pcb (KiCad board)
At the start: 2 copper layers, 80.5 x 60 mm, 15 parts, among them J1 Conn_01x04, J2_servo1 Conn_01x03, J4 Conn_01x03, U1 ESP32-WROOM-32

Commit message: updated PCB editor in KiCAD
Parts:
- moved R2_220Ω1 10.5 mm to (91.3, 127.0)
Routing:
- net GND: track 34.7 -> 127.8 mm, vias 0 -> 4
- net Net-(D1_GREEN1-A): track 0.00 -> 86.4 mm
- net Net-(U1-IO14): track 0.00 -> 84.0 mm
- net Net-(J2_servo1-Pin_2): track 0.00 -> 78.0 mm
- net Net-(J1-Pin_3): track 0.00 -> 64.6 mm
- net +5V: track 111.7 -> 176.2 mm
- net Net-(BZ1-+): track 0.00 -> 53.3 mm
- net Net-(D2_RED1-A): track 0.00 -> 52.0 mm
- net Net-(J1-Pin_2): track 0.00 -> 47.7 mm
- net Net-(U1-EN): track 0.00 -> 31.9 mm
